File: din_power_atm90e26.kicad_pcb (KiCad board)
At the start: 2 copper layers, 86.9 x 32.8 mm, 61 parts, among them J1 CONN_01X06, J2 VBAT, J3 CONN_01X08, J4 CONN_02X18, J5 CONN_01X08, U1 MCP73831-2-OT, U2 AP7365-33YG-13, U3 AP7365-33YG-13, U4 Hi-Link_SMPS, U5 dc-dc

Commit message: Add new part numbers and high voltage sym
Parts:
- added SYM1: SYM_Flash_Small, Whatnick_logo:Fsilk_HV, B.Cu at (132.3, 73.9)
Changed lines of the file:
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@@
     (tracks 770)
     (zones 0)
-    (modules 61)
+    (modules 62)
     (nets 56)
   )
@@
     (add_net VBAT)
   )
+  (module Whatnick_logo:Fsilk_HV (layer B.Cu)
+    (at 132.289 73.944 180)
+    (descr "Symbol, High Voltage, Type 2, Copper Top, Very Small,")
+    (tags "Symbol, High Voltage, Type 2, Copper Top, Very Small,")
+    (fp_text reference SYM1 (at -0.127 5.715 180) (layer B.SilkS) hide
+      (effects (font (size 1 1) (thickness 0.15)) (justify mirror))
+    )
+    (fp_text value SYM_Flash_Small (at -0.381 -4.572 180) (layer B.Fab)
+      (effects (font (size 1 1) (thickness 0.15)) (justify mirror))
+    )
+    (fp_line (start -4.699 -2.794) (end 0 4.191) (layer B.SilkS) (width 0.381))
+    (fp_line (start 4.699 -2.794) (end -4.699 -2.794) (layer B.SilkS) (width 0.381))
+    (fp_line (start 0 4.191) (end 4.699 -2.794) (layer B.SilkS) (width 0.381))
+    (fp_line (start -0.49784 -2.19964) (end -0.59944 -1.30048) (layer B.SilkS) (width 0.381))
+    (fp_line (start 0.29972 0.59944) (end -0.49784 -2.19964) (layer B.SilkS) (width 0.381))
+    (fp_line (start -0.89916 -0.20066) (end 0.29972 0.59944) (layer B.SilkS) (width 0.381))
+    (fp_line (start -0.09906 2.79908) (end -0.89916 -0.20066) (layer B.SilkS) (width 0.381))
+    (fp_line (start -0.49784 -2.19964) (end 0.1016 -1.50114) (layer B.SilkS) (width 0.381))
+    (fp_line (start -0.89916 -0.20066) (end 0.40132 2.60096) (layer B.SilkS) (width 0.381))
+    (fp_line (start 0.70104 0.89916) (end 0.1016 0.50038) (layer B.SilkS) (width 0.381))
+    (fp_line (start -0.49784 -2.19964) (end 0.70104 0.89916) (layer B.SilkS) (width 0.381))
+  )
   (module hi-link_smps:PCIE-36-SKT locked (layer B.Cu)

Commit message: Small silk screen changes and bump date
Other:
- board text added: "Whatnick Emon Base v1.2 07/12/2017"
- board text removed: "Whatnick Emon Base v1.2 06/12/2017"
Changed lines of the file:
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@@
     (37 F.SilkS user hide)
     (38 B.Mask user hide)
-    (39 F.Mask user)
+    (39 F.Mask user hide)
     (40 Dwgs.User user hide)
     (41 Cmts.User user hide)
     (42 Eco1.User user hide)
     (43 Eco2.User user hide)
-    (44 Edge.Cuts user)
+    (44 Edge.Cuts user hide)
     (45 Margin user hide)
     (46 B.CrtYd user hide)
-    (47 F.CrtYd user)
+    (47 F.CrtYd user hide)
     (48 B.Fab user hide)
     (49 F.Fab user hide)
@@
     (tags "capacitor 0603")
     (attr smd)
-    (fp_text reference C2 (at -2.168 -0.0394) (layer B.SilkS)
+    (fp_text reference C2 (at 2.12 0.032) (layer B.SilkS)
       (effects (font (size 0.5 0.5) (thickness 0.12)) (justify mirror))
     )
@@
     (tags "resistor 0603")
     (attr smd)
-    (fp_text reference R27 (at 2.295 -0.0156) (layer B.SilkS)
+    (fp_text reference R27 (at -2.247 -0.037) (layer B.SilkS)
       (effects (font (size 0.5 0.5) (thickness 0.12)) (justify mirror))
     )
@@
     (effects (font (size 1 1) (thickness 0.25)) (justify mirror))
   )
-  (gr_text "Whatnick Emon Base v1.2\n06/12/2017" (at 153.67 50.3174) (layer B.SilkS)
+  (gr_text "Whatnick Emon Base v1.2\n07/12/2017" (at 153.67 50.3174) (layer B.SilkS)
     (effects (font (size 1 1) (thickness 0.25)) (justify mirror))
   )

Commit message: New gerbers
Other:
- rule trace_min: 0.1 -> 0.2
Changed lines of the file:
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@@
   (page A4)
   (layers
-    (0 F.Cu signal hide)
-    (31 B.Cu signal hide)
-    (32 B.Adhes user hide)
-    (33 F.Adhes user hide)
-    (34 B.Paste user hide)
-    (35 F.Paste user hide)
+    (0 F.Cu signal)
+    (31 B.Cu signal)
+    (32 B.Adhes user)
+    (33 F.Adhes user)
+    (34 B.Paste user)
+    (35 F.Paste user)
     (36 B.SilkS user)
-    (37 F.SilkS user hide)
-    (38 B.Mask user hide)
-    (39 F.Mask user hide)
-    (40 Dwgs.User user hide)
-    (41 Cmts.User user hide)
-    (42 Eco1.User user hide)
-    (43 Eco2.User user hide)
-    (44 Edge.Cuts user hide)
-    (45 Margin user hide)
-    (46 B.CrtYd user hide)
-    (47 F.CrtYd user hide)
+    (37 F.SilkS user)
+    (38 B.Mask user)
+    (39 F.Mask user)
+    (40 Dwgs.User user)
+    (41 Cmts.User user)
+    (42 Eco1.User user)
+    (43 Eco2.User user)
+    (44 Edge.Cuts user)
+    (45 Margin user)
+    (46 B.CrtYd user)
+    (47 F.CrtYd user)
     (48 B.Fab user hide)
     (49 F.Fab user hide)
@@
     (zone_clearance 0.3)
     (zone_45_only yes)
-    (trace_min 0.1)
+    (trace_min 0.2)
     (segment_width 0.2)
     (edge_width 0.15)

Commit message: Update parts to fit Kicost
Parts:
- R14, R17, R7: value R -> 220K
- R33: value 470R -> 1K
Changed lines of the file:
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@@
       (effects (font (size 0.5 0.5) (thickness 0.12)) (justify mirror))
     )
-    (fp_text value R (at 0 -1.95 180) (layer B.Fab)
+    (fp_text value 220K (at 0 -1.95 180) (layer B.Fab)
       (effects (font (size 1 1) (thickness 0.15)) (justify mirror))
     )
@@
       (effects (font (size 0.5 0.5) (thickness 0.12)) (justify mirror))
     )
-    (fp_text value R (at 0 -1.95 180) (layer B.Fab)
+    (fp_text value 220K (at 0 -1.95 180) (layer B.Fab)
       (effects (font (size 1 1) (thickness 0.15)) (justify mirror))
     )
@@
       (effects (font (size 0.5 0.5) (thickness 0.12)))
     )
-    (fp_text value 470R (at 0 1.5) (layer F.Fab)
+    (fp_text value 1K (at 0 1.5) (layer F.Fab)
       (effects (font (size 1 1) (thickness 0.15)))
     )
@@
       (effects (font (size 0.5 0.5) (thickness 0.12)) (justify mirror))
     )
-    (fp_text value R (at 0 -1.95 180) (layer B.Fab)
+    (fp_text value 220K (at 0 -1.95 180) (layer B.Fab)
       (effects (font (size 1 1) (thickness 0.15)) (justify mirror))
     )
